Commit message: leaving tufts

File: kortex_description/robots/gen3_arm.urdf (robot description, URDF)
Before this commit: robot gen3, 11 links, 10 joints
Links:
- added link link4_col_link
Joints:
- added joint link4_col: type fixed, parent forearm_link, child link4_col_link, origin xyz=0 -0.1 0.0 rpy=0 0 0, axis 0 0 0
